Commit message: Get ros2 control working with ignition gazebo. Robot can be moved around by sending /cmd_vel

File: src/ground_bot1/description/robot.urdf.xacro (robot description, xacro)
@@ -2,3 +2,4 @@
 <robot xmlns:xacro="http://www.ros.org/wiki/xacro"  name="my_bot">
     <xacro:include filename="robot_core.xacro" />
+    <xacro:include filename="gazebo_control.xacro"/>
 </robot>

File: src/ground_bot1/description/robot_core.xacro (robot description, xacro)
@@ -37,5 +37,5 @@
             </geometry>
         </collision>
-        <xacro:inertial_box mass="0.5" x="0.3" y="0.3" z="0.15">
+        <xacro:inertial_box mass="2.0" x="0.3" y="0.3" z="0.15">
             <origin xyz="0.15 0 0.075" rpy="0 0 0"/>
         </xacro:inertial_box>
@@ -91,5 +91,5 @@
         <parent link="chassis"/>
         <child link="caster_wheel"/>
-        <origin xyz="0.24 0 0"/>
+        <origin xyz="0.25 0 0"/>
     </joint>
     <link name="caster_wheel">
@@ -104,4 +104,12 @@
                 <sphere radius="0.05"/>
             </geometry>
+            <surface>
+                <friction>
+                    <ode>
+                        <mu>0.0001</mu>  <!-- Higher friction coefficient -->
+                        <mu2>0.0001</mu2>  <!-- Friction in orthogonal direction -->
+                    </ode>
+                </friction>
+            </surface>
         </collision>
         <xacro:inertial_sphere mass="0.1" radius="0.05">

Commit message: Working Lidar model

File: src/ground_bot1/description/robot.urdf.xacro (robot description, xacro)
@@ -2,4 +2,5 @@
 <robot xmlns:xacro="http://www.ros.org/wiki/xacro"  name="my_bot">
     <xacro:include filename="robot_core.xacro" />
+    <xacro:include filename="lidar.xacro" />
     <xacro:include filename="gazebo_control.xacro"/>
 </robot>

File: src/ground_bot1/description/robot_core.xacro (robot description, xacro)
@@ -13,4 +13,7 @@
     <material name="black">
         <color rgba="0 0 0 1"/>
+    </material>
+    <material name="red">
+        <color rgba="1.0 0.2 0 1"/>
     </material>
     <!-- BASE LINK -->
@@ -37,5 +40,5 @@
             </geometry>
         </collision>
-        <xacro:inertial_box mass="2.0" x="0.3" y="0.3" z="0.15">
+        <xacro:inertial_box mass="5.0" x="0.3" y="0.3" z="0.15">
             <origin xyz="0.15 0 0.075" rpy="0 0 0"/>
         </xacro:inertial_box>
